File: keybored.kicad_pcb (KiCad board)
At the start: 2 copper layers, 316.7 x 133.3 mm, 161 parts, among them J1 USB_C_Receptacle_USB2.0, K1 KEYSW, K10 KEYSW, K11 KEYSW, K12 KEYSW, K13 KEYSW, K14 KEYSW, K15 KEYSW, K16 KEYSW, K17 KEYSW, K18 KEYSW, K19 KEYSW, K2 KEYSW, K20 KEYSW, K21 KEYSW, K22 KEYSW, K23 KEYSW, K24 KEYSW, K25 KEYSW, K26 KEYSW, K27 KEYSW, K28 KEYSW, K29 KEYSW, K3 KEYSW, K30 KEYSW, K31 KEYSW, K32 KEYSW, K33 KEYSW, K34 KEYSW, K35 KEYSW, K36 KEYSW, K37 KEYSW, K38 KEYSW, K39 KEYSW, K4 KEYSW, K40 KEYSW, K41 KEYSW, K43 KEYSW, K44 KEYSW, K45 KEYSW, K46 KEYSW, K47 KEYSW, K48 KEYSW, K49 KEYSW, K5 KEYSW, K50 KEYSW, K51 KEYSW, K52 KEYSW, K53 KEYSW, K54 KEYSW, K57 KEYSW, K58 KEYSW, K59 KEYSW, K6 KEYSW, K60 KEYSW, K61 KEYSW, K62 KEYSW, K63 KEYSW, K64 KEYSW, K65 KEYSW, K66 KEYSW, K67 KEYSW, K68 KEYSW, K69 KEYSW, K7 KEYSW, K8 KEYSW, K9 KEYSW, SW1 SW_PUSH, SW2 Rot_Enc_Sw, U1 ATMEGA32U4, U2 SSD1306-Display_Graphic, Y1 Crystal

Commit message: Major pcb changes
- now uses a dual footprint for switches
- added ARGB support
- added stabilizer holes
- added header pin support for ISP
Parts:
- removed K67, K68, K69: KEYSW, keyswitches:Kailh_socket_MX
- added D68: WS2812B, LED_SMD:LED_WS2812B_PLCC4_5.0x5.0mm_P3.2mm, B.Cu at (301.9, 98.7)
- added D69: WS2812B, LED_SMD:LED_WS2812B_PLCC4_5.0x5.0mm_P3.2mm, B.Cu at (244.3, 182.0)
- added D70: WS2812B, LED_SMD:LED_WS2812B_PLCC4_5.0x5.0mm_P3.2mm, B.Cu at (85.9, 142.6)
- added D72: WS2812B, LED_SMD:LED_WS2812B_PLCC4_5.0x5.0mm_P3.2mm, B.Cu at (343.1, 103.8)
- added D73: WS2812B, LED_SMD:LED_WS2812B_PLCC4_5.0x5.0mm_P3.2mm, B.Cu at (206.5, 182.2)
- added D74: WS2812B, LED_SMD:LED_WS2812B_PLCC4_5.0x5.0mm_P3.2mm, B.Cu at (87.5, 103.5)
- added D75: WS2812B, LED_SMD:LED_WS2812B_PLCC4_5.0x5.0mm_P3.2mm, B.Cu at (346.3, 142.6)
- added D76: WS2812B, LED_SMD:LED_WS2812B_PLCC4_5.0x5.0mm_P3.2mm, B.Cu at (174.6, 182.1)
- added D77: WS2812B, LED_SMD:LED_WS2812B_PLCC4_5.0x5.0mm_P3.2mm, B.Cu at (140.0, 103.5)
- added D78: WS2812B, LED_SMD:LED_WS2812B_PLCC4_5.0x5.0mm_P3.2mm, B.Cu at (328.5, 179.9)
- added D79: WS2812B, LED_SMD:LED_WS2812B_PLCC4_5.0x5.0mm_P3.2mm, B.Cu at (142.0, 182.1)
- added D80: WS2812B, LED_SMD:LED_WS2812B_PLCC4_5.0x5.0mm_P3.2mm, B.Cu at (192.4, 103.5)
- added D81: WS2812B, LED_SMD:LED_WS2812B_PLCC4_5.0x5.0mm_P3.2mm, B.Cu at (297.7, 179.9)
- added D82: WS2812B, LED_SMD:LED_WS2812B_PLCC4_5.0x5.0mm_P3.2mm, B.Cu at (86.4, 182.1)
- added D83: WS2812B, LED_SMD:LED_WS2812B_PLCC4_5.0x5.0mm_P3.2mm, B.Cu at (244.8, 103.6)
- added J2: ISP, Connector_PinHeader_2.54mm:PinHeader_2x03_P2.54mm_Vertical, F.Cu at (291.9, 84.0)
- added J3: RGB in, Connector_PinHeader_2.54mm:PinHeader_1x03_P2.54mm_Vertical, B.Cu at (311.1, 95.9)
- added J4: RGB out, Connector_PinHeader_2.54mm:PinHeader_1x03_P2.54mm_Vertical, B.Cu at (255.2, 99.3)
- added K42: KEYSW, keyswitches:Kailh_socket_MX_optional, F.Cu at (81.0, 171.4)
- added K55: KEYSW, keyswitches:Kailh_socket_MX_optional, F.Cu at (95.2, 190.5)
- added K56: KEYSW, keyswitches:Kailh_socket_MX_optional, F.Cu at (119.1, 190.5)
- added R7: 330, Resistor_SMD:R_0805_2012Metric_Pad1.15x1.40mm_HandSolder, F.Cu at (295.3, 100.2)
- added REF**: MountingHole_2.2mm_M2_Pad, MountingHole:MountingHole_2.2mm_M2_Pad, F.Cu at (61.9, 78.6)
- added REF**: MountingHole_2.2mm_M2_Pad, MountingHole:MountingHole_2.2mm_M2_Pad, F.Cu at (61.9, 102.4)
- added REF**: MountingHole_2.2mm_M2_Pad, MountingHole:MountingHole_2.2mm_M2_Pad, F.Cu at (369.1, 102.4)
- added REF**: MountingHole_2.2mm_M2_Pad, MountingHole:MountingHole_2.2mm_M2_Pad, F.Cu at (369.1, 78.6)
- added REF**: Stabilizer_MX_2u, keyswitches:Stabilizer_MX_2u, F.Cu at (81.0, 171.4)
- added REF**: Stabilizer_MX_2u, keyswitches:Stabilizer_MX_2u, F.Cu at (323.9, 152.4)
- added REF**: Stabilizer_MX_2u, keyswitches:Stabilizer_MX_2u, F.Cu at (326.2, 114.3)
- added REF**: MountingHole_2.2mm_M2_Pad, MountingHole:MountingHole_2.2mm_M2_Pad, F.Cu at (308.0, 122.0)
- added REF**: MountingHole_2.2mm_M2_Pad, MountingHole:MountingHole_2.2mm_M2_Pad, F.Cu at (308.0, 154.8)
- added REF**: MountingHole_2.2mm_M2_Pad, MountingHole:MountingHole_2.2mm_M2_Pad, F.Cu at (361.9, 173.8)
- added REF**: MountingHole_2.2mm_M2_Pad, MountingHole:MountingHole_2.2mm_M2_Pad, F.Cu at (309.6, 193.0)
- added REF**: MountingHole_2.2mm_M2_Pad, MountingHole:MountingHole_2.2mm_M2_Pad, F.Cu at (210.0, 193.0)
- added REF**: MountingHole_2.2mm_M2_Pad, MountingHole:MountingHole_2.2mm_M2_Pad, F.Cu at (135.7, 193.0)
- added REF**: MountingHole_2.2mm_M2_Pad, MountingHole:MountingHole_2.2mm_M2_Pad, F.Cu at (98.0, 173.8)
- added REF**: MountingHole_2.2mm_M2_Pad, MountingHole:MountingHole_2.2mm_M2_Pad, F.Cu at (86.0, 133.3)
- K1, K10, K11, K12, K13, K14, K15, K16, K17, K18, K19, K2, K20, K21, K22, K23, K24, K25, K26, K27, K28, K29, K3, K30, K31, K32, K33, K34, K35, K36, K37, K38, K39, K4, K40, K41, K43, K44, K45, K46, K47, K48, K49, K5, K50, K51, K52, K53, K54, K57, K58, K59, K6, K60, K61, K62, K63, K64, K65, K66, K7, K8, K9: footprint keyswitches:Kailh_socket_MX -> keyswitches:Kailh_socket_MX_optional
- moved K54 238.9 mm to (71.4, 190.5)
- moved K60 187.5 mm to (361.9, 114.3)
- moved K59 173.8 mm to (292.9, 190.5)
- moved K58 169.1 mm to (264.3, 190.5)
- moved K57 119.1 mm to (190.5, 190.5)
- moved K63 81.0 mm to (361.9, 195.3)
- moved K65 64.8 mm to (361.9, 133.3)
- moved K61 59.7 mm to (323.9, 195.3)
- moved K62 50.2 mm to (342.9, 195.3)
- moved K66 42.9 mm to (361.9, 152.4)
- moved K43 31.0 mm to (111.9, 171.4)
- moved K64 26.9 mm to (342.9, 176.2)
- moved K53 26.2 mm to (309.6, 171.4)
- moved K45 19.1 mm to (150.0, 171.4)
- moved K47 19.1 mm to (188.1, 171.4)
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- renumbered C6 to C1, C13 to C10, C4 to C11, C5 to C12, C7 to C2, C8 to C3, C9 to C4, C10 to C5, C1 to C6, C11 to C7, C2 to C8, C3 to C9, D43 to D42, D44 to D43, D45 to D44, D46 to D45, D47 to D46, D48 to D47, D49 to D48, D50 to D49, D51 to D50, D52 to D51, D53 to D52, D54 to D53, D57 to D54, D58 to D55, D59 to D56, D60 to D57, D61 to D58, D62 to D59, D63 to D60, D64 to D61, D65 to D62, D66 to D63, D67 to D64, D68 to D65, D69 to D66, D70 to D67, R9 to R10, R10 to R11, R7 to R8, R8 to R9
Connections:
- D42 pad 2: Net-(D43-Pad2) -> Net-(D42-Pad2)
- D43 pad 2: Net-(D44-Pad2) -> Net-(D43-Pad2)
- D44 pad 2: Net-(D45-Pad2) -> Net-(D44-Pad2)
- D45 pad 2: Net-(D46-Pad2) -> Net-(D45-Pad2)
- D46 pad 2: Net-(D47-Pad2) -> Net-(D46-Pad2)
- D47 pad 2: Net-(D48-Pad2) -> Net-(D47-Pad2)
- D48 pad 2: Net-(D49-Pad2) -> Net-(D48-Pad2)
- D49 pad 2: Net-(D50-Pad2) -> Net-(D49-Pad2)
- D50 pad 2: Net-(D51-Pad2) -> Net-(D50-Pad2)
- D51 pad 2: Net-(D52-Pad2) -> Net-(D51-Pad2)
- D52 pad 2: Net-(D53-Pad2) -> Net-(D52-Pad2)
- D53 pad 2: Net-(D54-Pad2) -> Net-(D53-Pad2)
- D54 pad 2: Net-(D57-Pad2) -> Net-(D54-Pad2)
- D55 pad 2: Net-(D58-Pad2) -> Net-(D55-Pad2)
- D56 pad 2: Net-(D59-Pad2) -> Net-(D56-Pad2)
- D57 pad 2: Net-(D60-Pad2) -> Net-(D57-Pad2)
- D58 pad 2: Net-(D61-Pad2) -> Net-(D58-Pad2)
- D59 pad 2: Net-(D62-Pad2) -> Net-(D59-Pad2)
- D60 pad 2: Net-(D63-Pad2) -> Net-(D60-Pad2)
- D61 pad 2: Net-(D64-Pad2) -> Net-(D61-Pad2)
- D62 pad 2: Net-(D65-Pad2) -> Net-(D62-Pad2)
- D63 pad 2: Net-(D66-Pad2) -> Net-(D63-Pad2)
- D64 pad 2: Net-(D67-Pad2) -> Net-(D64-Pad2)
- D65 pad 2: Net-(D68-Pad2) -> Net-(D65-Pad2)
- D66 pad 2: Net-(D69-Pad2) -> Net-(D66-Pad2)
- K49 pad 1: col6 -> col7
- K54 pad 1: col7 -> col8
- K61 pad 1: col8 -> col9
- K62 pad 1: col8 -> col9
- K63 pad 1: col8 -> col9
- U1 pad 1: Net-(U1-Pad1) -> RGB_IN
Routing:
- net VCC: track 152.9 -> 934.7 mm, vias 0 -> 3
- net Net-(D63-Pad2): track 23.9 -> 210.4 mm, vias 1 -> 0
- net Net-(D67-Pad2): track 162.3 -> 0.00 mm, vias 1 -> 0
- net Net-(D65-Pad2): track 186.6 -> 25.1 mm, vias 1 -> 0
- net Net-(D66-Pad2): track 193.1 -> 39.3 mm, vias 1 -> 0
- net Net-(D56-Pad2): track 0.00 -> 142.3 mm
- net col4: track 362.8 -> 500.4 mm
- net col2: track 340.8 -> 477.5 mm
- net col6: track 381.9 -> 515.4 mm
- net col8: track 444.8 -> 572.8 mm
- net Net-(D55-Pad2): track 0.00 -> 121.1 mm
- net col3: track 216.8 -> 336.2 mm
- net col0: track 244.1 -> 355.4 mm
- net col9: track 245.2 -> 355.9 mm
- net col7: track 236.2 -> 336.1 mm
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Other:
- board text added: "+5V"
- board text added: "Din"
- board text added: "Dout"
- board text added: "GND"
